File: board/avrg_board/FPGA.sch (KiCad schematic (older format))
At the start: 0 parts

Commit message: WIP: Add FPGA ports, Power labels, notes and comments
Parts:
- added U? (x8): ECP5U25-BG381, symbol ecp5:ECP5U25-BG381
Connections:
- new net GND: U?.B14 (GND[99]), U?.B7 (GND[99]), U?.C19 (GND[99]), U?.D4 (GND[99]), U?.F13 (GND[99]), U?.F14 (GND[99]), U?.F7 (GND[99]), U?.F8 (GND[99]), U?.G10 (GND[99]), U?.G11 (GND[99]), U?.G12 (GND[99]), U?.G13 (GND[99]), U?.G14 (GND[99]), U?.G15 (GND[99]), U?.G17 (GND[99]), U?.G4 (GND[99]), U?.G6 (GND[99]), U?.G7 (GND[99]), U?.G8 (GND[99]), U?.G9 (GND[99]), U?.H19 (GND[99]), U?.J10 (GND[99]), U?.J11 (GND[99]), U?.J12 (GND[99]), U?.J14 (GND[99]), U?.J2 (GND[99]), U?.J7 (GND[99]), U?.J9 (GND[99]), U?.K10 (GND[99]), U?.K11 (GND[99]), U?.K12 (GND[99]), U?.K14 (GND[99]), U?.K15 (GND[99]), U?.K6 (GND[99]), U?.K7 (GND[99]), U?.K9 (GND[99]), U?.L10 (GND[99]), U?.L11 (GND[99]), U?.L12 (GND[99]), U?.L9 (GND[99]), U?.M10 (GND[99]), U?.M11 (GND[99]), U?.M12 (GND[99]), U?.M14 (GND[99]), U?.M16 (GND[99]), U?.M2 (GND[99]), U?.M7 (GND[99]), U?.M9 (GND[99]), U?.N14 (GND[99]), U?.N15 (GND[99]), U?.N6 (GND[99]), U?.N7 (GND[99]), U?.P11 (GND[99]), U?.P12 (GND[99]), U?.P13 (GND[99]), U?.P14 (GND[99]), U?.P7 (GND[99]), U?.P8 (GND[99]), U?.R19 (GND[99]), U?.T10 (GND[99]), U?.T6 (GND[99]), U?.T7 (GND[99]), U?.T8 (GND[99]), U?.T9 (GND[99]), U?.U10 (GND[99]), U?.U11 (GND[99]), U?.U12 (GND[99]), U?.U13 (GND[99]), U?.U14 (GND[99]), U?.U6 (GND[99]), U?.U7 (GND[99]), U?.U8 (GND[99]), U?.U9 (GND[99]), U?.V10 (GND[99]), U?.V11 (GND[99]), U?.V12 (GND[99]), U?.V13 (GND[99]), U?.V14 (GND[99]), U?.V15 (GND[99]), U?.V16 (GND[99]), U?.V19 (GND[99]), U?.V20 (GND[99]), U?.V5 (GND[99]), U?.V6 (GND[99]), U?.V7 (GND[99]), U?.V8 (GND[99]), U?.V9 (GND[99]), U?.W12 (GND[99]), U?.W15 (GND[99]), U?.W16 (GND[99]), U?.W19 (GND[99]), U?.W6 (GND[99]), U?.W7 (GND[99]), U?.Y11 (GND[99]), U?.Y12 (GND[99]), U?.Y5 (GND[99]), U?.Y6 (GND[99]), U?.Y7 (GND[99]), U?.Y8 (GND[99])
- new net Vcc: U?.H10 (VCC[20]), U?.H11 (VCC[20]), U?.H12 (VCC[20]), U?.H13 (VCC[20]), U?.H8 (VCC[20]), U?.H9 (VCC[20]), U?.J13 (VCC[20]), U?.J8 (VCC[20]), U?.K13 (VCC[20]), U?.K8 (VCC[20]), U?.L13 (VCC[20]), U?.L8 (VCC[20]), U?.M13 (VCC[20]), U?.M8 (VCC[20]), U?.N10 (VCC[20]), U?.N11 (VCC[20]), U?.N12 (VCC[20]), U?.N13 (VCC[20]), U?.N8 (VCC[20]), U?.N9 (VCC[20])
- new net VccAux: U?.F15 (VCCAUX[4]), U?.F6 (VCCAUX[4]), U?.P15 (VCCAUX[4]), U?.P6 (VCCAUX[4])
- new net VccIO_0: U?.F10 (VCCIO0[2]), U?.F9 (VCCIO0[2])
- new net VccIO_1: U?.F11 (VCCIO1[2]), U?.F12 (VCCIO1[2])
- new net VccIO_2: U?.H14 (VCCIO2[3]), U?.H15 (VCCIO2[3]), U?.J15 (VCCIO2[3])
- new net VccIO_3: U?.L14 (VCCIO3[3]), U?.L15 (VCCIO3[3]), U?.M15 (VCCIO3[3])
- new net VccIO_6: U?.L6 (VCCIO6[3]), U?.L7 (VCCIO6[3]), U?.M6 (VCCIO6[3])
- new net VccIO_7: U?.H6 (VCCIO7[3]), U?.H7 (VCCIO7[3]), U?.J6 (VCCIO7[3])
- new net VccIO_8: U?.P10 (VCCIO8[2]), U?.P9 (VCCIO8[2])
Other:
- note added: "Only A and B have true LVDS.\nEmulated need termination resistors.\nTN1262\n"
Changed lines of the file:
@@
 EESchema Schematic File Version 4
+LIBS:avrg_board-cache
 EELAYER 29 0
 EELAYER END
 $Descr A4 11693 8268
 encoding utf-8
-Sheet 1 10
+Sheet 7 11
 Title ""
 Date ""
@@
 Comment4 ""
 $EndDescr
+$Comp
+L ecp5:ECP5U25-BG381 U?
+U 1 1 5CF8EB97
+P 1400 700
+F 0 "U?" H 2530 -397 60  0000 L CNN
+F 1 "ECP5U25-BG381" H 2530 -503 60  0000 L CNN
+F 2 "" H 1400 700 50  0001 C CNN
+F 3 "" H 1400 700 50  0001 C CNN
+	1    1400 700
+	1    0    0    -1
+$EndComp
+$Comp
+L ecp5:ECP5U25-BG381 U?
+U 2 1 5CF973E8
+P 4200 700
+F 0 "U?" H 5330 -797 60  0000 L CNN
+F 1 "ECP5U25-BG381" H 5330 -903 60  0000 L CNN
+F 2 "" H 4200 700 50  0001 C CNN
+F 3 "" H 4200 700 50  0001 C CNN
+	2    4200 700
+	1    0    0    -1
+$EndComp
+$Comp
+L ecp5:ECP5U25-BG381 U?
+U 3 1 5CFA0EBA
+P 7300 700
+F 0 "U?" H 8430 -797 60  0000 L CNN
+F 1 "ECP5U25-BG381" H 8430 -903 60  0000 L CNN
+F 2 "" H 7300 700 50  0001 C CNN
+F 3 "" H 7300 700 50  0001 C CNN
+	3    7300 700
+	1    0    0    -1
+$EndComp
+$Comp
+L ecp5:ECP5U25-BG381 U?
+U 4 1 5CFA736B
+P 9800 700
+F 0 "U?" H 10700 -2700 60  0000 L CNN
+F 1 "ECP5U25-BG381" H 10200 -2600 60  0000 L CNN
+F 2 "" H 9800 700 50  0001 C CNN
+F 3 "" H 9800 700 50  0001 C CNN
+	4    9800 700
+	1    0    0    -1
+$EndComp
+$Comp
+L ecp5:ECP5U25-BG381 U?
+U 5 1 5CFB435A
+P 1300 4100
+F 0 "U?" H 2630 2603 60  0000 L CNN
+F 1 "ECP5U25-BG381" H 2630 2497 60  0000 L CNN
+F 2 "" H 1300 4100 50  0001 C CNN
+F 3 "" H 1300 4100 50  0001 C CNN
+	5    1300 4100
+	1    0    0    -1
+$EndComp
+$Comp
+L ecp5:ECP5U25-BG381 U?
+U 6 1 5CFB96E3
+P 4200 4100
+F 0 "U?" H 5330 2603 60  0000 L CNN
+F 1 "ECP5U25-BG381" H 5330 2497 60  0000 L CNN
+F 2 "" H 4200 4100 50  0001 C CNN
+F 3 "" H 4200 4100 50  0001 C CNN
+	6    4200 4100
+	1    0    0    -1
+$EndComp
+$Comp
+L ecp5:ECP5U25-BG381 U?
+U 7 1 5CFC0CEC
+P 6900 4100
+F 0 "U?" H 8730 3003 60  0000 L CNN
+F 1 "ECP5U25-BG381" H 8730 2897 60  0000 L CNN
+F 2 "" H 6900 4100 50  0001 C CNN
+F 3 "" H 6900 4100 50  0001 C CNN
+	7    6900 4100
+	1    0    0    -1
+$EndComp
+$Comp
+L ecp5:ECP5U25-BG381 U?
+U 8 1 5CFC96B5
+P 10300 5000
+F 0 "U?" H 10500 5300 60  0000 L CNN
+F 1 "ECP5U25-BG381" H 10400 5200 60  0000 L CNN
+F 2 "" H 10300 5000 50  0001 C CNN
+F 3 "" H 10300 5000 50  0001 C CNN
+	8    10300 5000
+	1    0    0    -1
+$EndComp
+Text Notes 600  3700 0    118  ~ 0
+Only A and B have true LVDS.\nEmulated need termination resistors.\nTN1262\n
+Text GLabel 10300 5200 0    50   Input ~ 0
+VccIO_0
+Text GLabel 10300 5300 0    50   Input ~ 0
+VccIO_1
+Text GLabel 10300 5400 0    50   Input ~ 0
+VccIO_2
+Text GLabel 10300 5500 0    50   Input ~ 0
+VccIO_3
+Text GLabel 10300 5600 0    50   Input ~ 0
+VccIO_6
+Text GLabel 10300 5700 0    50   Input ~ 0
+VccIO_7
+Text GLabel 10300 5800 0    50   Input ~ 0
+VccIO_8
+$Comp
+L power:GND #PWR?
+U 1 1 5D6150E1
+P 10300 5000
+F 0 "#PWR?" H 10300 4750 50  0001 C CNN
+F 1 "GND" V 10305 4872 50  0000 R CNN
+F 2 "" H 10300 5000 50  0001 C CNN
+F 3 "" H 10300 5000 50  0001 C CNN
+	1    10300 5000
+	0    1    1    0
+$EndComp
+Text GLabel 10300 5900 0    50   Input ~ 0
+Vcc
+Text GLabel 10300 5100 0    50   Input ~ 0
+VccAux
 $EndSCHEMATC
