File: board/avrg_board/IO.sch (KiCad schematic (older format))
At the start: 0 parts

Commit message: WIP: Add FPGA ports, Power labels, notes and comments
Other:
- note added: "LEDS\nButtons\nDisplay\nSensors?\nDUAL PMOD\nGPIO with level converters\nGPIO without level converters\nDifferential pairs\ntype of connectors?"
Changed lines of the file:
@@
 EESchema Schematic File Version 4
+LIBS:avrg_board-cache
 EELAYER 29 0
 EELAYER END
 $Descr A4 11693 8268
 encoding utf-8
-Sheet 1 10
+Sheet 9 11
 Title ""
 Date ""
@@
 Comment4 ""
 $EndDescr
+Text Notes 3400 3950 0    118  ~ 0
+LEDS\nButtons\nDisplay\nSensors?\nDUAL PMOD\nGPIO with level converters\nGPIO without level converters\nDifferential pairs\ntype of connectors?
 $EndSCHEMATC
