File: board/avrg_board/JTAG.sch (KiCad schematic (older format))
At the start: 0 parts

Commit message: WIP: Add FPGA ports, Power labels, notes and comments
Parts:
- added J?: Conn_01x06, symbol Connector_Generic:Conn_01x06
- added R? (x10): 4k7, symbol Device:R
- added R? (x2): 1k, symbol Device:R
- added SW?: SW_DIP_x03, symbol Switch:SW_DIP_x03
Connections:
- new net CCLK: R?.2
- new net CFG_0: R?.2, SW?.6
- new net CFG_1: R?.2, SW?.5
- new net CFG_2: R?.2, SW?.4
- new net CSSPIN: R?.2
- new net GND: J?.6 (Pin_6), R?.1, SW?.1, SW?.2, SW?.3
- new net INITN: R?.2
- new net MCLK: R?.2
- new net PROGRAMN: R?.2
- new net TCK: J?.5 (Pin_5), R?.2
- new net TDI: J?.2 (Pin_2), R?.2
- new net TDO: J?.4 (Pin_4), R?.2
- new net TMS: J?.3 (Pin_3), R?.2
- new net VccIO_8: J?.1 (Pin_1), R?.1, R?.1, R?.1, R?.1, R?.1, R?.1, R?.1, R?.1, R?.1, R?.1, R?.1
Other:
- note added: "CFG PINS\n"
- note added: "JTAG"
