File: board/avrg_board/SERDES.sch (KiCad schematic (older format))
At the start: 0 parts

Commit message: WIP: Add FPGA ports, Power labels, notes and comments
Other:
- note added: "USB 3.0?\nGigabit Ethernet ?\nPCI Express 2.0 ?\nSMA connectors?\n"
Changed lines of the file:
@@
 EESchema Schematic File Version 4
+LIBS:avrg_board-cache
 EELAYER 29 0
 EELAYER END
 $Descr A4 11693 8268
 encoding utf-8
-Sheet 1 1
+Sheet 11 11
 Title ""
 Date ""
@@
 Comment4 ""
 $EndDescr
+Text Notes 4000 2200 0    118  ~ 0
+USB 3.0?\nGigabit Ethernet ?\nPCI Express 2.0 ?\nSMA connectors?\n
 $EndSCHEMATC
