File: board/avrg_board/SPI.sch (KiCad schematic (older format))
At the start: 0 parts

Commit message: WIP: Add FPGA ports, Power labels, notes and comments
Parts:
- added J?: Micro_SD_Card_Det, symbol Connector:Micro_SD_Card_Det
Other:
- note added: "on borad spi flash?\n"
Changed lines of the file:
@@
 EESchema Schematic File Version 4
+LIBS:avrg_board-cache
 EELAYER 29 0
 EELAYER END
 $Descr A4 11693 8268
 encoding utf-8
-Sheet 1 10
+Sheet 10 11
 Title ""
 Date ""
@@
 Comment4 ""
 $EndDescr
+$Comp
+L Connector:Micro_SD_Card_Det J?
+U 1 1 5D64BB5D
+P 2150 1650
+F 0 "J?" H 2100 2467 50  0000 C CNN
+F 1 "Micro_SD_Card_Det" H 2100 2376 50  0000 C CNN
+F 2 "" H 4200 2350 50  0001 C CNN
+F 3 "https://www.hirose.com/product/en/download_file/key_name/DM3/category/Catalog/doc_file_id/49662/?file_category_id=4&item_id=195&is_series=1" H 2150 1750 50  0001 C CNN
+	1    2150 1650
+	1    0    0    -1
+$EndComp
+Text Notes 4400 1900 0    118  ~ 0
+on borad spi flash?\n
 $EndSCHEMATC
