File: board/avrg_board/UART.sch (KiCad schematic (older format))
At the start: 0 parts

Commit message: WIP: Add FPGA ports, Power labels, notes and comments
Parts:
- added P?: USB_C_Plug_USB2.0, symbol Connector:USB_C_Plug_USB2.0
Connections:
- new net: P?.A1 (GND), P?.A12 (GND), P?.B1 (GND), P?.B12 (GND)
- new net: P?.A4 (VBUS), P?.A9 (VBUS), P?.B4 (VBUS), P?.B9 (VBUS)
Other:
- note added: "FTDI chip\n"
- note added: "USB2.0 but with 3.0 enclosure\n"
Changed lines of the file:
@@
 EESchema Schematic File Version 4
+LIBS:avrg_board-cache
 EELAYER 29 0
 EELAYER END
 $Descr A4 11693 8268
 encoding utf-8
-Sheet 1 10
+Sheet 8 11
 Title ""
 Date ""
@@
 Comment4 ""
 $EndDescr
+$Comp
+L Connector:USB_C_Plug_USB2.0 P?
+U 1 1 5D64C1F5
+P 7750 2300
+F 0 "P?" H 7857 3167 50  0000 C CNN
+F 1 "USB_C_Plug_USB2.0" H 7857 3076 50  0000 C CNN
+F 2 "" H 7900 2300 50  0001 C CNN
+F 3 "https://www.usb.org/sites/default/files/documents/usb_type-c.zip" H 7900 2300 50  0001 C CNN
+	1    7750 2300
+	1    0    0    -1
+$EndComp
+Text Notes 7450 1300 0    118  ~ 0
+USB2.0 but with 3.0 enclosure\n
+Text Notes 3650 1950 0    118  ~ 0
+FTDI chip\n
 $EndSCHEMATC
