File: board/avrg_board/clock.sch (KiCad schematic (older format))
At the start: 0 parts

Commit message: WIP: Add FPGA ports, Power labels, notes and comments
Other:
- note added: "High speed I/O can be used as clock input. \nTake care of possible noise. read TN1265"
Changed lines of the file:
@@
 EESchema Schematic File Version 4
+LIBS:avrg_board-cache
 EELAYER 29 0
 EELAYER END
 $Descr A4 11693 8268
 encoding utf-8
-Sheet 1 10
+Sheet 3 11
 Title ""
 Date ""
@@
 Comment4 ""
 $EndDescr
+Text Notes 3000 1800 0    118  ~ 0
+High speed I/O can be used as clock input.  \nTake care of possible noise. read TN1265
 $EndSCHEMATC
