File: board/avrg_board/memory.sch (KiCad schematic (older format))
At the start: 0 parts

Commit message: WIP: Add FPGA ports, Power labels, notes and comments
Other:
- note added: "Look TN1265 high-speed I/O\n\n\nHyperram?\nDDR3?\nDDR2?\nFlash?"
Changed lines of the file:
@@
 EESchema Schematic File Version 4
+LIBS:avrg_board-cache
 EELAYER 29 0
 EELAYER END
 $Descr A4 11693 8268
 encoding utf-8
-Sheet 1 10
+Sheet 4 11
 Title ""
 Date ""
@@
 Comment4 ""
 $EndDescr
+Text Notes 3900 2250 0    118  ~ 0
+Look TN1265 high-speed I/O\n\n\nHyperram?\nDDR3?\nDDR2?\nFlash?
 $EndSCHEMATC
