File: board/avrg_board/video.sch (KiCad schematic (older format))
At the start: 0 parts

Commit message: WIP: Add FPGA ports, Power labels, notes and comments
Parts:
- added J?: DB15_Male_HighDensity, symbol Connector:DB15_Male_HighDensity
Other:
- note added: "HDMI ?\nVGA?\nDVI?\n"
Changed lines of the file:
@@
 EESchema Schematic File Version 4
+LIBS:avrg_board-cache
 EELAYER 29 0
 EELAYER END
 $Descr A4 11693 8268
 encoding utf-8
-Sheet 1 10
+Sheet 6 11
 Title ""
 Date ""
@@
 Comment4 ""
 $EndDescr
+$Comp
+L Connector:DB15_Male_HighDensity J?
+U 1 1 5D55B1FE
+P 1750 1700
+F 0 "J?" H 1750 2567 50  0000 C CNN
+F 1 "DB15_Male_HighDensity" H 1750 2476 50  0000 C CNN
+F 2 "" H 800 2100 50  0001 C CNN
+F 3 " ~" H 800 2100 50  0001 C CNN
+	1    1750 1700
+	1    0    0    -1
+$EndComp
+Text Notes 3600 1750 0    118  ~ 0
+HDMI ?\nVGA?\nDVI?\n
 $EndSCHEMATC
